Commit message: Adding initial rework of surus. It is properly facing the correct direction (visually) where the front of the robot is facing towards the x axis. The left actuator is also now setup with the prismatic joint to the upper assembly. Next commit will be with right actuator. Need to look into how to control joint position for actuator as it seems that ros control cant directly be used in a sdf file, but instead a urdf file where a transmission tag is inserted

File: surus_sim/robots/surus_sim.URDF (robot description, URDF)
Before this commit: robot surus_sim, 16 links, 15 joints
Links:
- removed link left_front_wheel
- removed link left_mid_wheel
- removed link left_vert_back_link
- removed link left_vert_front_link
- removed link rear_left_wheel_link
- removed link rear_right_wheel
- removed link right_front_wheel
- removed link right_mid_wheel
- removed link right_vert_back_link
- removed link right_vert_front_link
- added link Upper_link, mass 6.26524835038105; collision mesh filename=package://surus_sim/meshes/Upper_link.STL; visual mesh filename=package://surus_sim/meshes/Upper_link.STL
- added link bl_wheel_link, mass 0.891962924275681; collision mesh filename=package://surus_sim/meshes/bl_wheel_link.STL; visual mesh filename=package://surus_sim/meshes/bl_wheel_link.STL
- added link br_wheel_link, mass 0.891962924275675; collision mesh filename=package://surus_sim/meshes/br_wheel_link.STL; visual mesh filename=package://surus_sim/meshes/br_wheel_link.STL
- added link left_actuator_pivot_link, mass 0.310659429014437; collision mesh filename=package://surus_sim/meshes/left_actuator_pivot_link.STL; visual mesh filename=package://surus_sim/meshes/left_actuator_pivot_link.STL
- added link left_actuator_shaft_link, mass 0.132261419151138; collision mesh filename=package://surus_sim/meshes/left_actuator_shaft_link.STL; visual mesh filename=package://surus_sim/meshes/left_actuator_shaft_link.STL
- added link left_back_bot_vert_link, mass 0.322840822636628; collision mesh filename=package://surus_sim/meshes/left_back_bot_vert_link.STL; visual mesh filename=package://surus_sim/meshes/left_back_bot_vert_link.STL
- added link left_front_bot_vert_link, mass 0.224203755199739; collision mesh filename=package://surus_sim/meshes/left_front_bot_vert_link.STL; visual mesh filename=package://surus_sim/meshes/left_front_bot_vert_link.STL
- added link left_front_wheel_link, mass 0.828510835025874; collision mesh filename=package://surus_sim/meshes/left_front_wheel_link.STL; visual mesh filename=package://surus_sim/meshes/left_front_wheel_link.STL
- added link left_mid_wheel_link, mass 0.82851083502594; collision mesh filename=package://surus_sim/meshes/left_mid_wheel_link.STL; visual mesh filename=package://surus_sim/meshes/left_mid_wheel_link.STL
- added link right_actuator_base_link, mass 0.310659429014436; collision mesh filename=package://surus_sim/meshes/right_actuator_base_link.STL; visual mesh filename=package://surus_sim/meshes/right_actuator_base_link.STL
- added link right_actuator_shaft_link, mass 0.132261419151135; collision mesh filename=package://surus_sim/meshes/right_actuator_shaft_link.STL; visual mesh filename=package://surus_sim/meshes/right_actuator_shaft_link.STL
- added link right_back_bot_vert_link, mass 0.322840822636629; collision mesh filename=package://surus_sim/meshes/right_back_bot_vert_link.STL; visual mesh filename=package://surus_sim/meshes/right_back_bot_vert_link.STL
- added link right_front_bot_vert_link, mass 0.32284082263663; collision mesh filename=package://surus_sim/meshes/right_front_bot_vert_link.STL; visual mesh filename=package://surus_sim/meshes/right_front_bot_vert_link.STL
- added link right_front_wheel_link, mass 0.828510835025939; collision mesh filename=package://surus_sim/meshes/right_front_wheel_link.STL; visual mesh filename=package://surus_sim/meshes/right_front_wheel_link.STL
- added link right_middle_wheel_link, mass 0.828510835025941; collision mesh filename=package://surus_sim/meshes/right_middle_wheel_link.STL; visual mesh filename=package://surus_sim/meshes/right_middle_wheel_link.STL
- link base_link: mass 4.88149894403649 -> 4.66238075193942
- link left_bot_link: mass 0.431669670198118 -> 0.426568340691013
- link left_top_link: mass 0.221531862132748 -> 0.219608847869789
- link rear_rocker_link: mass 0.765248646616661 -> 0.68717511332603
- link right_bot_link: mass 0.431669670198118 -> 0.433325599142795
- link right_top_link: mass 0.221531862132748 -> 0.215121814589556
Joints:
- removed joint left_top_link_joint
- removed joint left_vert_back_top_joint
- removed joint left_vert_front_top_joint
- removed joint mid_wheel_joint
- removed joint rear_left_wheel_joint
- removed joint rear_right_wheel_joint
- removed joint right_vert_top_back_joint
- removed joint right_vert_top_front_joint
- added joint Upper_joint: type fixed, parent base_link, child Upper_link, origin xyz=0.350126900454533 -0.167586499483468 0.248709793231653 rpy=1.5707963267949 0.000586226261771362 0, axis 0 0 0
- added joint bl_wheel_joint: type continuous, parent rear_rocker_link, child bl_wheel_link, origin xyz=-0.0252750000000036 0.353962500000001 -0.138937999999999 rpy=0 0 0, axis 0 1 0
- added joint br_wheel_joint: type continuous, parent rear_rocker_link, child br_wheel_link, origin xyz=-0.0255249999999962 -0.3539625 -0.138938000000001 rpy=0 0 0, axis 0 -1 0
- added joint left_actuator_pivot_joint: type continuous, parent base_link, child left_actuator_pivot_link, origin xyz=-0.250185317620025 0.215890000516527 0.138937085309467 rpy=0 0 0, axis 0 1 0
- added joint left_actuator_top_pivot_joint: type continuous, parent Upper_link, child left_actuator_shaft_link, origin xyz=-0.190676873416691 0.324089724612332 -0.402716999999999 rpy=-1.5707963267949 8.52587309432495E-15 0.816085048104826, axis 0 1 0
- added joint left_back_bot_vert_joint: type continuous, parent left_bot_link, child left_back_bot_vert_link, origin xyz=-0.1778 0.00317499999999793 0 rpy=0 0 0, axis 0 -1 0
- added joint left_front_bot_vert_joint: type continuous, parent left_bot_link, child left_front_bot_vert_link, origin xyz=0.1778 -0.00158749999999819 0 rpy=0 0 0, axis 0 -1 0
- added joint left_top_joint: type continuous, parent base_link, child left_top_link, origin xyz=0.178439682379975 0.220652500516531 0.215137085309467 rpy=0 0 0, axis 0 1 0
- added joint right_actuator_top_pivot_joint: type continuous, parent Upper_link, child right_actuator_shaft_link, origin xyz=-0.190676873416686 0.324089724612333 0.0720598000000012 rpy=-1.5707963267949 8.68206969619894E-15 0.816085048104826, axis 0 -1 0
- added joint right_back_bot_vert_joint: type continuous, parent right_bot_link, child right_back_bot_vert_link, origin xyz=-0.1778 0.00634999999999813 0 rpy=0 0 0, axis 0 -1 0
- added joint right_front_bot_vert_joint: type continuous, parent right_bot_link, child right_front_bot_vert_link, origin xyz=0.177958749596813 0.00633000103306119 0 rpy=0 0 0, axis 0 -1 0
- added joint right_middle_wheel_joint: type continuous, parent right_back_bot_vert_link, child right_middle_wheel_link, origin xyz=-0.000457386250926561 -0.14015 -0.138937303366726 rpy=0 0 0, axis 0 -1 0
- added joint roght_actuator_base_joint: type continuous, parent base_link, child right_actuator_base_link, origin xyz=0.159640049698826 -0.239646299483471 0.572911241939758 rpy=-4.92623675962194E-15 -0.815498821843055 6.76618012987679E-15, axis 0 -1 0
- joint left_bot_joint: axis 0 0 -1 -> 0 1 0; origin xyz=-0.20638 0.18733 0.004986 rpy=-1.5708 -6.123E-17 -1.5708 -> xyz=0.178621978509024 0.220652500516531 0.138937303366726 rpy=0 0 0
- joint left_front_wheel_joint: axis 0 0 -1 -> 0 1 0; child left_front_wheel -> left_front_wheel_link; origin xyz=-0.19888 0.072035 -0.02585 rpy=0 0 1.179 -> xyz=0.000457386250926506 0.135387500000001 -0.138937303366725 rpy=0 0 0; parent left_vert_front_link -> left_front_bot_vert_link
- joint left_mid_wheel_joint: axis 0 0 1 -> 0 1 0; child left_mid_wheel -> left_mid_wheel_link; origin xyz=0.198883561596939 -0.0820347706495037 -0.0258499999996897 rpy=3.14159265358979 0 -2.78551494975313 -> xyz=0 0.130644998966941 -0.138938169159622 rpy=0 0 0; parent left_vert_back_link -> left_back_bot_vert_link
- joint rear_rocker_joint: origin xyz=0 -0.31433 0.004986 rpy=-1.5708 -6.123E-17 -1.5708 -> xyz=-0.313685317620023 0 0.138937085309467 rpy=0 0 0
- joint right_bot_joint: axis 0 0 -1 -> 0 -1 0; origin xyz=0.206375 0.187325 0.014986 rpy=1.5707963267949 6.12303176911189E-17 1.5707963267949 -> xyz=0.17825738625093 -0.220672499483469 0.138937303366725 rpy=0 0 0
- joint right_front_wheel_joint: axis 0 0 -1 -> 0 -1 0; child right_front_wheel -> right_front_wheel_link; origin xyz=0.000125000000000042 0.205138 0.0258499999996902 rpy=0 0 3.14159265358979 -> xyz=-0.000167933171141499 -0.14015 -0.138937954740417 rpy=0 0 0; parent right_vert_front_link -> right_front_bot_vert_link
- joint right_top_joint: axis 0 0 -1 -> 0 -1 0; origin xyz=0.206375 0.18732500000002 0.0811859999999602 rpy=-1.5707963267949 -6.12303176911189E-17 -1.5707963267949 -> xyz=0.17843968237998 -0.220672499483469 0.215137085309466 rpy=0 0 0

Commit message: Added ros_control support for left and right actuators. Need to load the URDF of the robot AS WELL AS the sdf in order for ros_control to read the <transmission> tags from the URDF.

File: surus_sim/robots/surus_sim.URDF (robot description, URDF)
Before this commit: robot surus_sim, 21 links, 20 joints
Links:
- removed link left_actuator_pivot_link
- removed link left_actuator_shaft_link
- removed link right_actuator_base_link
- removed link right_actuator_shaft_link
- added link left_bot_actuator_link, mass 0.310659429014436; collision mesh filename=package://rmc_simulation/surus_sim/meshes/left_bot_actuator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; visual mesh filename=package://rmc_simulation/surus_sim/meshes/left_bot_actuator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
- added link left_top_actuator_link, mass 0.132261419151138; collision mesh filename=package://rmc_simulation/surus_sim/meshes/left_top_actuator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; visual mesh filename=package://rmc_simulation/surus_sim/meshes/left_top_actuator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
- added link right_bot_actuator_link, mass 0.310659429014436; collision mesh filename=package://rmc_simulation/surus_sim/meshes/right_bot_actuato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; visual mesh filename=package://rmc_simulation/surus_sim/meshes/right_bot_actuato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
- added link right_top_actuator_link, mass 0.132261419151135; collision mesh filename=package://rmc_simulation/surus_sim/meshes/right_top_actuato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; visual mesh filename=package://rmc_simulation/surus_sim/meshes/right_top_actuato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
- link Upper_link: geometry collision mesh filename=package://rmc_simulation/surus_sim/meshes/Upper_link.STL; visual mesh filename=package://rmc_simulation/surus_sim/meshes/Upper_link.STL
- link base_link: geometry collision mesh filename=package://rmc_simulation/surus_sim/meshes/base_link.STL; visual mesh filename=package://rmc_simulation/surus_sim/meshes/base_link.STL
- link bl_wheel_link: mass 0.891962924275681 -> 0.89196292427568; geometry collision mesh filename=package://rmc_simulation/surus_sim/meshes/bl_wheel_link.STL; visual mesh filename=package://rmc_simulation/surus_sim/meshes/bl_wheel_link.STL
- link br_wheel_link: geometry collision mesh filename=package://rmc_simulation/surus_sim/meshes/br_wheel_link.STL; visual mesh filename=package://rmc_simulation/surus_sim/meshes/br_wheel_link.STL
- link left_back_bot_vert_link: geometry collision mesh filename=package://rmc_simulation/surus_sim/meshes/left_back_bot_ver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; visual mesh filename=package://rmc_simulation/surus_sim/meshes/left_back_bot_ver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
- link left_bot_link: geometry collision mesh filename=package://rmc_simulation/surus_sim/meshes/left_bot_link.STL; visual mesh filename=package://rmc_simulation/surus_sim/meshes/left_bot_link.STL
- link left_front_bot_vert_link: geometry collision mesh filename=package://rmc_simulation/surus_sim/meshes/left_front_bot_ve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; visual mesh filename=package://rmc_simulation/surus_sim/meshes/left_front_bot_ve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
- link left_front_wheel_link: geometry collision mesh filename=package://rmc_simulation/surus_sim/meshes/left_front_wheel_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; visual mesh filename=package://rmc_simulation/surus_sim/meshes/left_front_wheel_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
- link left_mid_wheel_link: mass 0.82851083502594 -> 0.828510835025941; geometry collision mesh filename=package://rmc_simulation/surus_sim/meshes/left_mid_wheel_li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; visual mesh filename=package://rmc_simulation/surus_sim/meshes/left_mid_wheel_li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
- link left_top_link: mass 0.219608847869789 -> 0.21960884786979; geometry collision mesh filename=package://rmc_simulation/surus_sim/meshes/left_top_link.STL; visual mesh filename=package://rmc_simulation/surus_sim/meshes/left_top_link.STL
- link rear_rocker_link: geometry collision mesh filename=package://rmc_simulation/surus_sim/meshes/rear_rocker_link.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; visual mesh filename=package://rmc_simulation/surus_sim/meshes/rear_rocker_link.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
- link right_back_bot_vert_link: geometry collision mesh filename=package://rmc_simulation/surus_sim/meshes/right_back_bot_ve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; visual mesh filename=package://rmc_simulation/surus_sim/meshes/right_back_bot_ve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
- link right_bot_link: geometry collision mesh filename=package://rmc_simulation/surus_sim/meshes/right_bot_link.STL; visual mesh filename=package://rmc_simulation/surus_sim/meshes/right_bot_link.STL
- link right_front_bot_vert_link: geometry collision mesh filename=package://rmc_simulation/surus_sim/meshes/right_front_bot_v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; visual mesh filename=package://rmc_simulation/surus_sim/meshes/right_front_bot_v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
- link right_front_wheel_link: mass 0.828510835025939 -> 0.828510835025938; geometry collision mesh filename=package://rmc_simulation/surus_sim/meshes/right_front_wheel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; visual mesh filename=package://rmc_simulation/surus_sim/meshes/right_front_wheel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
- link right_middle_wheel_link: geometry collision mesh filename=package://rmc_simulation/surus_sim/meshes/right_middle_whee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; visual mesh filename=package://rmc_simulation/surus_sim/meshes/right_middle_whee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
- link right_top_link: geometry collision mesh filename=package://rmc_simulation/surus_sim/meshes/right_top_link.STL; visual mesh filename=package://rmc_simulation/surus_sim/meshes/right_top_link.STL
Joints:
- removed joint left_actuator_pivot_joint
- removed joint left_actuator_top_pivot_joint
- removed joint right_actuator_top_pivot_joint
- removed joint roght_actuator_base_joint
- added joint left_mid_actuator_joint: type prismatic, parent left_top_actuator_link, child left_bot_actuator_link, origin xyz=-0.5588 -0.010351 0 rpy=0 0 -3.9443E-31, axis -1 0 0, limit lower=0 upper=0.4572 effort=100.0 velocity=0.1
- added joint left_top_actuator_joint: type continuous, parent Upper_link, child left_top_actuator_link, origin xyz=0.624074367318843 0.235140500000006 0.031384156630293 rpy=-4.7603420685916E-15 -0.815498821843055 6.53832397580358E-15, axis 0 1 0
- added joint right_mid_actuator_joint: type prismatic, parent right_top_actuator_link, child right_bot_actuator_link, origin xyz=-0.5588 0.0148462999999999 0 rpy=3.94430452610506E-31 0 3.94430452610506E-31, axis -1 0 0, limit lower=0 upper=0.4572 effort=100.0 velocity=0.1
- added joint right_top_actuator_joint: type continuous, parent Upper_link, child right_top_actuator_link, origin xyz=0.62407 -0.23964 0.031384 rpy=-4.9262E-15 -0.8155 6.7662E-15, axis 0 -1 0
- joint Upper_joint: axis 0 0 0 -> 0 -1 0; origin xyz=0.350126900454533 -0.167586499483468 0.248709793231653 rpy=1.5707963267949 0.000586226261771362 0 -> xyz=-0.464434317620022 0 0.541527085309466 rpy=0 0 0; type fixed -> continuous

Commit message: Readding blackfly mount link so I can now work on panning search for aruco marker

File: surus_sim/robots/surus_sim.URDF (robot description, URDF)
Before this commit: robot surus_sim, 21 links, 20 joints
Joints:
- joint left_mid_actuator_joint: limit lower=0 upper=0.4572 effort=100.0 velocity=0.1 -> lower=0 upper=1.4 effort=100.0 velocity=0.2
- joint right_mid_actuator_joint: limit lower=0 upper=0.4572 effort=100.0 velocity=0.1 -> lower=0 upper=1.4 effort=100.0 velocity=0.2

Commit message: Adding equivalent links to those in the SDF so that robot_state_publisher can take care of broadcasting sensor transforms for the most part and allow arbotix to control the joint state of the servo joint in the URDF. This will need to move to the rmc_software repo and should be inside a surus_description package

File: surus_sim/robots/surus_sim.URDF (robot description, URDF)
Before this commit: robot surus_sim, 21 links, 20 joints
Links:
- removed link Upper_link
- removed link bl_wheel_link
- removed link br_wheel_link
- removed link left_back_bot_vert_link
- removed link left_bot_actuator_link
- removed link left_bot_link
- removed link left_front_bot_vert_link
- removed link left_front_wheel_link
- removed link left_mid_wheel_link
- removed link left_top_actuator_link
- removed link left_top_link
- removed link rear_rocker_link
- removed link right_back_bot_vert_link
- removed link right_bot_actuator_link
- removed link right_bot_link
- removed link right_front_bot_vert_link
- removed link right_front_wheel_link
- removed link right_middle_wheel_link
- removed link right_top_actuator_link
- removed link right_top_link
- added link blackfly_mount_link, mass 1e5; collision box size=0.05 0.05 0.05; visual box size=0.05 0.05 0.05
- added link blackfly_optical_link
- added link imu, mass 1e5
- added link servo_mount_link, mass 1e5
- link base_link: mass 4.66238075193942 -> None; geometry visual mesh filename=package://rmc_simulation/surus_sim/meshes/visual_meshes/bas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
Joints:
- removed joint Upper_joint
- removed joint bl_wheel_joint
- removed joint br_wheel_joint
- removed joint left_back_bot_vert_joint
- removed joint left_bot_joint
- removed joint left_front_bot_vert_joint
- removed joint left_front_wheel_joint
- removed joint left_mid_actuator_joint
- removed joint left_mid_wheel_joint
- removed joint left_top_actuator_joint
- removed joint left_top_joint
- removed joint rear_rocker_joint
- removed joint right_back_bot_vert_joint
- removed joint right_bot_joint
- removed joint right_front_bot_vert_joint
- removed joint right_front_wheel_joint
- removed joint right_mid_actuator_joint
- removed joint right_middle_wheel_joint
- removed joint right_top_actuator_joint
- removed joint right_top_joint
- added joint blackfly_mount_joint: type continuous, parent servo_mount_link, child blackfly_mount_link, origin xyz=0 0 0.051 rpy=0 0 3.14159, axis 0 0 1
- added joint blackfly_optical_joint: type fixed, parent blackfly_mount_link, child blackfly_optical_link, origin xyz=0 0 0 rpy=-1.57 0 -1.57, axis 0 0 1
- added joint imu_joint: type fixed, parent base_link, child imu, origin xyz=0.1 -0.3 0 rpy=0 0 0, axis 0 0 1
- added joint servo_mount_joint: type fixed, parent base_link, child servo_mount_link, origin xyz=-0.30 -0.40 0.4191 rpy=0 0 0, axis 0 0 1

Commit message: Changed rotation of camera mounted on servo. This will need to get correct to 0 yaw for blackfly_mount_joint when sumanth mills a new mounting plate

File: surus_sim/robots/surus_sim.URDF (robot description, URDF)
Before this commit: robot surus_sim, 5 links, 4 joints
Joints:
- joint blackfly_mount_joint: origin xyz=0 0 0.051 rpy=0 0 3.14159 -> xyz=0 0 0.051 rpy=0 0 -1.57
- joint imu_joint: origin xyz=0.1 -0.3 0 rpy=0 0 0 -> xyz=-0.05 0.14 0 rpy=0 0 0

Commit message: Fixed simulation to work with current sensor_integrated work

File: surus_sim/robots/surus_sim.URDF (robot description, URDF)
Before this commit: robot surus_sim, 5 links, 4 joints
Joints:
- joint blackfly_mount_joint: origin xyz=0 0 0.051 rpy=0 0 -1.57 -> xyz=0 0 0.051 rpy=0 0 0
- joint servo_mount_joint: origin xyz=-0.30 -0.40 0.4191 rpy=0 0 0 -> xyz=-0.30 -0.40 0.4191 rpy=0 0 3.14159
